File: orthgyle.kicad_pcb (KiCad board)
At the start: 2 copper layers, 357.8 x 95.2 mm, 198 parts, among them J1 USB, J2 AVR_ISP_6, U1 ATMEGA328-PU, Y1 16MHz

Commit message: Update PCB page settings
Parts:
- moved BOOT1 74.7 mm to (384.9, 103.0)
- moved C12 74.7 mm to (369.7, 98.2)
- moved C14 74.7 mm to (371.0, 175.4)
- moved D40 74.7 mm to (384.9, 151.6)
- moved D45 74.7 mm to (384.9, 162.0)
- moved D54 74.7 mm to (373.5, 162.0)
- moved D58 74.7 mm to (373.5, 151.6)
- moved D78 74.7 mm to (357.6, 104.0)
- moved D79 74.7 mm to (357.6, 123.0)
- moved D80 74.7 mm to (357.6, 142.0)
- moved D82 74.7 mm to (357.6, 180.0)
- moved RESET1 74.7 mm to (384.9, 98.2)
- moved Y1 74.7 mm to (384.9, 117.8)
- moved D50 74.7 mm to (384.9, 172.5)
- moved D70 74.7 mm to (373.5, 172.5)
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
Commit message: Flip 2u stabilizers
Parts:
- MX30_2u1, MX50_2u1: footprint Orthgyle:MX_PCB_200B -> Orthgyle:MX_PCB_200H

Commit message: Move decoupling capacitors closer to ICs
Parts:
- moved D30 326.4 mm to (39.2, 151.6)
- moved C5 325.1 mm to (383.6, 123.2), turned to -90 degrees
- moved D25 323.1 mm to (39.2, 162.0)
- moved C4 314.2 mm to (367.8, 118.8), turned to 90 degrees
- moved D71 55.2 mm to (385.0, 162.0)
- moved C8 37.8 mm to (63.8, 149.1), turned to -90 degrees
- moved C12 33.9 mm to (357.7, 129.9), turned to -90 degrees
- moved C7 28.7 mm to (63.8, 130.0), turned to -90 degrees
- moved C13 26.9 mm to (357.7, 148.9), turned to -90 degrees
- moved D40 21.0 mm to (385.0, 172.5)
- moved D15 21.0 mm to (36.3, 151.6)
- moved C9 19.9 mm to (63.7, 168.0), turned to -90 degrees
- moved C15 17.5 mm to (362.1, 175.3)
- moved C14 15.2 mm to (357.7, 168.0), turned to -90 degrees
- moved C11 13.8 mm to (357.7, 111.3), turned to -90 degrees
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Routing:
- net Net-(D25-A): track 210.3 -> 131.9 mm
- net Net-(D71-K): track 25.7 -> 98.2 mm
- net Net-(D30-A): track 203.6 -> 161.1 mm
- net +5V: track 651.3 -> 689.7 mm
- net /ROW0: track 424.3 -> 452.4 mm
- net Net-(D5-A): track 70.4 -> 47.8 mm
- net Net-(D26-A): track 128.8 -> 147.9 mm
- net /ROW3: track 430.6 -> 415.1 mm, vias 0 -> 1
- net Net-(D31-A): track 163.5 -> 148.5 mm
- net Net-(D10-A): track 89.9 -> 77.0 mm
- net /RESET: track 52.8 -> 65.5 mm
- net Net-(D15-A): track 94.3 -> 106.2 mm
- net Net-(D36-K): track 187.2 -> 176.6 mm
- net Net-(D40-K): track 188.5 -> 178.1 mm
- net Net-(D1-A): track 32.0 -> 21.9 mm
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