File: orthgyle.kicad_pcb (KiCad board)
At the start: 2 copper layers, 357.8 x 95.2 mm, 198 parts, among them J1 USB, J2 AVR_ISP_6, U1 ATMEGA328-PU, Y1 16MHz

Commit message: Rename RGB diodes
Parts:
- added J3: JST, Connector_JST:JST_SH_SM04B-SRSS-TB_1x04-1MP_P1.00mm_Horizontal, F.Cu at (3.92, 3.31)
- renumbered D78 to RGB1, D87 to RGB10, D79 to RGB2, D80 to RGB3, D81 to RGB4, D82 to RGB5, D83 to RGB6, D84 to RGB7, D85 to RGB8, D86 to RGB9
Routing:
- net Net-(D76-K): track 43.3 -> 44.3 mm
- net Net-(J1-CC2): vias 1 -> 0
Other:
- board text added: "Orthgyle rev1 Jan 2025"
- board text removed: "Orthgyle rev1 Dec 2024"

Commit message: Align USB port with case location
Switch to SK6812 mini-e LEDs
Flip stabilizer orientation
Parts:
- removed C12, C13, C14, C8, C9: 1uF, Capacitor_THT:C_Disc_D4.3mm_W1.9mm_P5.00mm
- removed the C7 at (63.8, 130.0)
- removed J3: JST, Connector_JST:JST_SH_SM04B-SRSS-TB_1x04-1MP_P1.00mm_Horizontal
- added ST62: 7U, Orthgyle:MX-7U-Stabilizer, F.Cu at (210.6, 180.1)
- MX30_2u1, MX50_2u1: footprint Orthgyle:MX_PCB_200H -> Orthgyle:MX_PCB_200
- MX40: footprint Orthgyle:MX_PCB_700H -> Orthgyle:MX
- RGB1, RGB10, RGB2, RGB3, RGB4, RGB5, RGB6, RGB7, RGB8, RGB9: footprint LED_SMD:LED_WS2812B_PLCC4_5.0x5.0mm_P3.2mm -> Orthgyle:SK6812-MINI-E; moved to B.Cu
- moved C6 13.0 mm to (361.9, 99.1), turned to 0 degrees
- moved C4 12.7 mm to (59.2, 99.1), turned to 180 degrees
- moved D76 3.69 mm to (41.9, 127.6)
- moved D77 3.69 mm to (41.9, 130.5)
- moved C3 3.69 mm to (44.9, 122.9)
- moved F1 2.02 mm to (43.1, 105.8)
- moved LED1 1.67 mm to (46.2, 138.6)
- moved J1 1.07 mm to (44.9, 96.0)
- moved RGB10 0.71 mm to (63.0, 103.6), turned to -90 degrees
- moved RGB1 0.71 mm to (358.1, 103.6)
- moved RGB9 0.69 mm to (63.0, 122.9), turned to -90 degrees
- moved RGB6 0.69 mm to (63.0, 180.0), turned to -90 degrees
- moved RGB7 0.69 mm to (63.0, 161.0), turned to -90 degrees
- moved RGB8 0.69 mm to (63.0, 142.0), turned to -90 degrees
- moved RGB2 0.59 mm to (358.1, 122.9)
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- renumbered C6 to C4, C10 to C5, C11 to C6, C15 to C7
Routing:
- net +5V: track 689.7 -> 621.9 mm, vias 0 -> 3
- net Net-(RGB10-DIN): track 26.3 -> 14.8 mm
- net Net-(RGB7-DOUT): track 26.0 -> 14.5 mm
- net Net-(RGB6-DOUT): track 26.0 -> 14.5 mm
- net Net-(RGB8-DOUT): track 25.9 -> 14.7 mm
- net /LED1: track 367.0 -> 375.8 mm
- net /ROW2: track 428.2 -> 436.9 mm
- net Net-(D2-A): track 54.6 -> 62.5 mm
- net /COL4: track 414.6 -> 421.3 mm, vias 0 -> 1
- net /LED2: track 40.4 -> 46.9 mm
- net Net-(D36-K): track 176.6 -> 182.9 mm
- net Net-(RGB5-DOUT): track 303.5 -> 297.8 mm
- net Net-(D37-K): track 188.5 -> 194.1 mm
- net Net-(D47-K): track 125.9 -> 131.0 mm
- net /COL5: track 399.2 -> 404.2 mm
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Other:
- board text added: "A5"
- board text added: "A8"
- board text added: "D+"
- board text added: "D-"
- board text added: "GND"
- board text added: "ISP"
- board text added: "Orthgyle rev 2 Feb 2025"
- board text added: "VCC"
- board text removed: "Orthgyle rev1 Jan 2025"

Commit message: Switch LEDs to SK6812-mini-e
Parts:
- renumbered C4 to C6, C6 to C7, C5 to C8, C7 to C9
Other:
- board text added: "Orthgyle rev2"
- board text removed: "Orthgyle rev 2 Feb 2025"
