File: orthgyle.kicad_pcb (KiCad board)
At the start: 2 copper layers, 357.8 x 95.2 mm, 193 parts, among them J1 USB, J2 AVR_ISP_6, U1 ATMEGA328-PU, Y1 16MHz

Commit message: Add center offset 2u keys
Parts:
- removed ST62: 7U, Orthgyle:MX-7U-Stabilizer
- added J3: Conn_02x01, Jumper:SolderJumper-2_P1.3mm_Bridged_RoundedPad1.0x1.5mm, B.Cu at (38.6, 102.9)
- added J4: Conn_02x01, Jumper:SolderJumper-2_P1.3mm_Bridged_RoundedPad1.0x1.5mm, B.Cu at (48.8, 102.9)
- added J5: Conn_02x01, Jumper:SolderJumper-2_P1.3mm_Bridged_RoundedPad1.0x1.5mm, B.Cu at (41.1, 102.9)
- added J6: Conn_02x01, Jumper:SolderJumper-2_P1.3mm_Bridged_RoundedPad1.0x1.5mm, B.Cu at (46.2, 102.9)
- added J7: Conn_02x01, Jumper:SolderJumper-2_P1.3mm_Bridged_RoundedPad1.0x1.5mm, B.Cu at (43.7, 102.9)
- added J8: Conn_02x01, Jumper:SolderJumper-2_P1.3mm_Bridged_RoundedPad1.0x1.5mm, B.Cu at (51.3, 102.9)
- added MX35_2: SW_Push, Orthgyle:MX_PCB_200H, F.Cu at (182.0, 180.1)
- added MX45_2: SW_Push, Orthgyle:MX_PCB_200H, F.Cu at (239.2, 180.1)
- MX30_2: renamed from MX30_2u1; footprint Orthgyle:MX_PCB_200 -> Orthgyle:MX_PCB_200H
- MX40: footprint Orthgyle:MX -> Orthgyle:MX_PCB_700H
- MX50_2: renamed from MX50_2u1; footprint Orthgyle:MX_PCB_200 -> Orthgyle:MX_PCB_200H
Connections:
- F1 pad 1: Net-(F1-Pad1) -> Net-(J3-Pin_2)
- J1 pad A4: Net-(F1-Pad1) -> Net-(J3-Pin_1)
- J1 pad A6: Net-(D76-K) -> Net-(J7-Pin_1)
- J1 pad A7: Net-(D77-K) -> Net-(J6-Pin_1)
- J1 pad A9: Net-(F1-Pad1) -> Net-(J3-Pin_1)
- J1 pad B4: Net-(F1-Pad1) -> Net-(J3-Pin_1)
- J1 pad B6: Net-(D76-K) -> Net-(J7-Pin_1)
- J1 pad B7: Net-(D77-K) -> Net-(J6-Pin_1)
- J1 pad B9: Net-(F1-Pad1) -> Net-(J3-Pin_1)
- R5 pad 2: Net-(J1-CC1) -> Net-(J4-Pin_2)
- R6 pad 2: Net-(J1-CC2) -> Net-(J5-Pin_2)
Routing:
- net Net-(J4-Pin_2): track 0.00 -> 18.5 mm, vias 0 -> 1
- net Net-(J1-CC1): track 24.0 -> 6.20 mm, vias 0 -> 1
- net Net-(J3-Pin_1): track 0.00 -> 14.9 mm, vias 0 -> 1
- net Net-(J5-Pin_2): track 0.00 -> 14.5 mm
- net /COL1: track 453.1 -> 466.5 mm
- net Net-(J1-CC2): track 19.0 -> 5.60 mm, vias 0 -> 1
- net Net-(F1-Pad1): track 12.8 -> 0.00 mm
- net /COL6: track 366.1 -> 375.7 mm
- net Net-(D35-A): track 172.2 -> 181.7 mm
- net Net-(D76-K): track 43.4 -> 34.0 mm, vias 1 -> 0
- net Net-(D77-K): track 51.1 -> 42.5 mm, vias 2 -> 0
- net Net-(J6-Pin_1): track 0.00 -> 8.52 mm, vias 0 -> 1
- net Net-(J7-Pin_1): track 0.00 -> 6.88 mm, vias 0 -> 1
- net Net-(J3-Pin_2): track 0.00 -> 5.48 mm
- net GND: track 1.45 -> 6.89 mm
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